Commit message: Update to new sonar image format

File: urdf/es200-7c.urdf (robot description, URDF)
Before this commit: robot simrad_es200-7c, 2 links, 1 joints
Links:
- link ek80_nav: geometry 

Commit message: Many updates

File: urdf/es200-7c.urdf (robot description, URDF)
Before this commit: robot simrad_es200-7c, 2 links, 1 joints
Links:
- removed link ek80_nav
- added link ek80_nav_level
Joints:
- joint nav_to_transducer: origin rpy=0 1.57075 0 -> rpy=3.1415 0 0; parent ek80_nav -> ek80_nav_level
